Commit message: Change tsukuba2022 to igvc2023

File: igvc2023/urdf/sensors/hokuyo.urdf.xacro (robot description, xacro)
@@ -21,5 +21,5 @@
         <origin xyz="0 0 0" rpy="0 0 0"/>
         <geometry>
-          <mesh filename="package://tsukuba2022/meshes/hokuyo.dae"/>
+          <mesh filename="package://igvc2023/meshes/hokuyo.dae"/>
         </geometry>
       </visual>
