Commit message: Change gps position

File: igvc2023/urdf/sensors/gps.urdf.xacro (robot description, xacro)
@@ -12,5 +12,5 @@
     <link name="${name}_link">
       <visual>
-        <origin xyz="0.2 0 0" rpy="0 0 0"/>
+        <origin xyz="1 0 0" rpy="0 0 0"/>
         <geometry>
           <sphere radius="0.015"/>
@@ -18,5 +18,5 @@
       </visual>
       <collision>
-        <origin xyz="0 0 0" rpy="0 0 0"/>
+        <origin xyz="1 0 0" rpy="0 0 0"/>
         <geometry>
           <sphere radius="0.015"/>
