Commit message: Change tsukuba2022 to igvc2023

File: igvc2023/urdf/orange2022.xacro (robot description, xacro)
@@ -16,17 +16,17 @@
   </xacro:macro>
   <!-- Import gazebo reference -->
-  <xacro:include filename="$(find tsukuba2022)/urdf/orange2022.gazebo"/>
+  <xacro:include filename="$(find igvc2023)/urdf/orange2022.gazebo"/>
   <!-- Import 2D LiDAR model -->
-  <xacro:include filename="$(find tsukuba2022)/urdf/sensors/hokuyo.urdf.xacro"/>
+  <xacro:include filename="$(find igvc2023)/urdf/sensors/hokuyo.urdf.xacro"/>
   <xacro:sensor_hokuyo name="hokuyo" parent="base_link" min_angle="-1.22" max_angle="1.22" samples="720">
     <origin xyz="0.1075 0.0 0.1085" rpy="0.0 0.0 0.0"/>
   </xacro:sensor_hokuyo>
   <!-- Import 3D LiDAR model -->
-  <xacro:include filename="$(find tsukuba2022)/urdf/sensors/velodyne.urdf.xacro"/>
+  <xacro:include filename="$(find igvc2023)/urdf/sensors/velodyne.urdf.xacro"/>
   <xacro:sensor_velodyne name="velodyne" parent="base_link" min_angle="-2.35619" max_angle="2.35619" samples="720">
     <origin xyz="-0.0185 0.0 0.8985" rpy="0.0 0.0 0.0"/>
   </xacro:sensor_velodyne>
   <!-- Import imu model -->
-  <xacro:include filename="$(find tsukuba2022)/urdf/sensors/imu.urdf.xacro"/>
+  <xacro:include filename="$(find igvc2023)/urdf/sensors/imu.urdf.xacro"/>
   <xacro:sensor_imu name="imu" parent="base_link" size="0.05 0.05 0.05">
     <origin xyz="-0.253 0.0 0.068" rpy="0.0 0.0 0.0"/>
@@ -50,5 +50,5 @@
       <origin xyz="0.0775 0.25275 0.6425" rpy="0.0 0.0 0.0"/>
       <geometry>
-        <mesh filename="package://tsukuba2022/meshes/chassis.dae"/>
+        <mesh filename="package://igvc2023/meshes/chassis.dae"/>
       </geometry>
     </visual>
@@ -80,5 +80,5 @@
       <origin xyz="-0.4815 0.145 -0.039" rpy="0.0 0.0 0.0"/>
       <geometry>
-        <mesh filename="package://tsukuba2022/meshes/left_back_wheel.dae"/>
+        <mesh filename="package://igvc2023/meshes/left_back_wheel.dae"/>
       </geometry>
     </visual>
@@ -94,5 +94,5 @@
       <origin xyz="-0.4815 -0.145 -0.039" rpy="0.0 0.0 0.0"/>
       <geometry>
-        <mesh filename="package://tsukuba2022/meshes/right_back_wheel.dae"/>
+        <mesh filename="package://igvc2023/meshes/right_back_wheel.dae"/>
         <sphere radius="0.0625"/>
       </geometry>
@@ -124,5 +124,5 @@
       <origin xyz="0.0 0.0 0.0" rpy="0.0 0.0 0.0"/>
       <geometry>
-        <mesh filename="package://tsukuba2022/meshes/front_wheel.dae"/>
+        <mesh filename="package://igvc2023/meshes/front_wheel.dae"/>
       </geometry>
     </visual>
@@ -143,5 +143,5 @@
       <origin xyz="0.0 0.0 0.0" rpy="0.0 0.0 0.0"/>
       <geometry>
-        <mesh filename="package://tsukuba2022/meshes/front_wheel.dae"/>
+        <mesh filename="package://igvc2023/meshes/front_wheel.dae"/>
       </geometry>
     </visual>

File: igvc2023/urdf/sensors/velodyne.urdf.xacro (robot description, xacro)
@@ -21,5 +21,5 @@
         <origin xyz="0 0 0" rpy="0 0 0"/>
         <geometry>
-          <mesh filename="package://tsukuba2022/meshes/velodyne.dae"/>
+          <mesh filename="package://igvc2023/meshes/velodyne.dae"/>
         </geometry>
       </visual>

Commit message: Add camera urdf

File: igvc2023/urdf/orange2022.xacro (robot description, xacro)
@@ -32,4 +32,9 @@
     <origin xyz="-0.253 0.0 0.068" rpy="0.0 0.0 0.0"/>
   </xacro:sensor_imu>
+  <!-- Import fisheye camera model -->
+  <xacro:include filename="$(find igvc2023)/urdf/sensors/camera.urdf.xacro"/>
+  <xacro:sensor_camera name="camera" parent="base_link">
+    <origin xyz="0 0 1.3" rpy="0 ${PI/2} 0"/>
+  </xacro:sensor_camera>
   <!-- Base Footprint -->
   <joint name="base_joint" type="fixed">

Commit message: add GPS

File: igvc2023/urdf/orange2022.xacro (robot description, xacro)
@@ -37,4 +37,9 @@
     <origin xyz="0 0 1.3" rpy="0 ${PI/2} 0"/>
   </xacro:sensor_camera>
+  <!-- Import fisheye gps model -->
+  <xacro:include filename="$(find igvc2023)/urdf/sensors/gps.urdf.xacro"/>
+  <xacro:sensor_gps name="gps" parent="base_link">
+    <origin xyz="0.1 0 1.0" rpy="0 0 0"/>
+  </xacro:sensor_gps>
   <!-- Base Footprint -->
   <joint name="base_joint" type="fixed">
