Commit message: add GPS

File: igvc2023/urdf/orange.xacro (robot description, xacro)
@@ -37,4 +37,8 @@
     <origin xyz="0 0 1.3" rpy="0 ${PI/2} 0"/>
   </xacro:sensor_camera>
+  <xacro:include filename="$(find igvc2023)/urdf/sensors/gps.urdf.xacro"/>
+  <xacro:sensor_gps name="gps" parent="base_link">
+    <origin xyz="0 0 1.3" rpy="0 ${PI} 0"/>
+  </xacro:sensor_gps>
   <!-- Base Footprint -->
   <joint name="base_joint" type="fixed">

Commit message: add GPS

File: igvc2023/urdf/orange.xacro (robot description, xacro)
@@ -37,4 +37,9 @@
     <origin xyz="0 0 1.3" rpy="0 ${PI/2} 0"/>
   </xacro:sensor_camera>
+  <!-- Import fisheye camera model -->
+  <xacro:include filename="$(find igvc2023)/urdf/sensors/gps.urdf.xacro"/>
+  <xacro:sensor_gps name="gps" parent="base_link">
+    <origin xyz="0 0.2 1" rpy="0 ${PI} 0"/>
+  </xacro:sensor_gps>
   <!-- Base Footprint -->
   <joint name="base_joint" type="fixed">

Commit message: fix gps position

File: igvc2023/urdf/orange.xacro (robot description, xacro)
@@ -40,5 +40,5 @@
   <xacro:include filename="$(find igvc2023)/urdf/sensors/gps.urdf.xacro"/>
   <xacro:sensor_gps name="gps" parent="base_link">
-    <origin xyz="0 0.2 1" rpy="0 ${PI} 0"/>
+    <origin xyz="0 0 1" rpy="0 ${PI} 0"/>
   </xacro:sensor_gps>
   <!-- Base Footprint -->

File: igvc2023/urdf/sensors/gps.urdf.xacro (robot description, xacro)
@@ -12,5 +12,5 @@
     <link name="${name}_link">
       <visual>
-        <origin xyz="0 0 0" rpy="0 0 0"/>
+        <origin xyz="0.2 0 0" rpy="0 0 0"/>
         <geometry>
           <sphere radius="0.015"/>

Commit message: Change orange.xacro

File: igvc2023/urdf/orange.xacro (robot description, xacro)
@@ -20,20 +20,20 @@
   <xacro:include filename="$(find igvc2023)/urdf/sensors/hokuyo.urdf.xacro"/>
   <xacro:sensor_hokuyo name="hokuyo" parent="base_link" min_angle="-1.22" max_angle="1.22" samples="720">
-    <origin xyz="0.1075 0.0 0.1085" rpy="0.0 0.0 0.0"/>
+    <origin xyz="0.2875 0.0 0.1085" rpy="0.0 0.0 0.0"/>
   </xacro:sensor_hokuyo>
   <!-- Import 3D LiDAR model -->
   <xacro:include filename="$(find igvc2023)/urdf/sensors/velodyne.urdf.xacro"/>
   <xacro:sensor_velodyne name="velodyne" parent="base_link" min_angle="-2.35619" max_angle="2.35619" samples="720">
-    <origin xyz="-0.0185 0.0 0.8985" rpy="0.0 0.0 0.0"/>
+    <origin xyz="-0.25 0.0 1.25" rpy="0.0 0.0 0.0"/>
   </xacro:sensor_velodyne>
   <!-- Import imu model -->
   <xacro:include filename="$(find igvc2023)/urdf/sensors/imu.urdf.xacro"/>
   <xacro:sensor_imu name="imu" parent="base_link" size="0.05 0.05 0.05">
-    <origin xyz="-0.253 0.0 0.068" rpy="0.0 0.0 0.0"/>
+    <origin xyz="0 0.0 0.068" rpy="0.0 0.0 0.0"/>
   </xacro:sensor_imu>
   <!-- Import fisheye camera model -->
   <xacro:include filename="$(find igvc2023)/urdf/sensors/camera.urdf.xacro"/>
   <xacro:sensor_camera name="camera" parent="base_link">
-    <origin xyz="0 0 1.3" rpy="0 ${PI/2} 0"/>
+    <origin xyz="-0.25 0 1.6" rpy="0 ${PI/2} 0"/>
   </xacro:sensor_camera>
   <!-- Import gps model -->
@@ -52,19 +52,19 @@
   <link name="base_link">
     <collision>
-      <origin xyz="-0.1995 0.0 0.341" rpy="0.0 0.0 0.0"/>
+      <origin xyz="-0.6 0.0 0.5" rpy="0.0 0.0 0.0"/>
       <geometry>
-        <box size="0.549 0.5055 0.603"/>
+        <box size="1.06 0.625 0.83"/>
       </geometry>
     </collision>
     <visual>
-      <origin xyz="0.0775 0.25275 0.6425" rpy="0.0 0.0 0.0"/>
+      <origin xyz="-0.6 0.0 0.5" rpy="0.0 0.0 0.0"/>
       <geometry>
-        <mesh filename="package://igvc2023/meshes/chassis.dae"/>
+        <mesh filename="package://igvc2023/meshes/IGVCchassis.dae"/>
       </geometry>
     </visual>
     <inertial>
-       <mass value="27.1" />
-       <origin xyz="-0.1995 0.0 0.19" rpy="0.0 0.0 0.0"/>
-       <xacro:box_inertia m="27.1" x="0.549" y="0.5055" z="0.3"/>
+       <mass value="40" />
+       <origin xyz="-0.6 0.0 0.3" rpy="0.0 0.0 0.0"/>
+       <xacro:box_inertia m="40" x="1.06" y="0.625" z="0.43"/>
     </inertial>
   </link>
@@ -82,5 +82,5 @@
   <link name="left_caster_link">
     <collision>
-      <origin xyz="-0.4815 0.145 -0.039" rpy="0.0 ${PI/2} ${PI/2}"/>
+      <origin xyz="-1.28015 0.15 -0.039" rpy="0.0 ${PI/2} ${PI/2}"/>
       <geometry>
         <sphere radius="0.0625"/>
@@ -88,5 +88,5 @@
     </collision>
     <visual>
-      <origin xyz="-0.4815 0.145 -0.039" rpy="0.0 0.0 0.0"/>
+      <origin xyz="-1.2015 0.15 -0.039" rpy="0.0 0.0 0.0"/>
       <geometry>
         <mesh filename="package://igvc2023/meshes/left_back_wheel.dae"/>
@@ -96,5 +96,5 @@
   <link name="right_caster_link">
     <collision>
-      <origin xyz="-0.4815 -0.145 -0.039" rpy="0.0 ${PI/2} ${PI/2}"/>
+      <origin xyz="-1.2015 -0.15 -0.039" rpy="0.0 ${PI/2} ${PI/2}"/>
       <geometry>
         <sphere radius="0.0625"/>
@@ -102,5 +102,5 @@
     </collision>
     <visual>
-      <origin xyz="-0.4815 -0.145 -0.039" rpy="0.0 0.0 0.0"/>
+      <origin xyz="-1.2015 -0.15 -0.039" rpy="0.0 0.0 0.0"/>
       <geometry>
         <mesh filename="package://igvc2023/meshes/right_back_wheel.dae"/>
@@ -111,5 +111,5 @@
   <!-- Front wheels -->
   <joint type="revolute" name="left_wheel_hinge">
-    <origin xyz="0.0 0.2834 0.0" rpy="0.0 0.0 0.0"/>
+    <origin xyz="0.0 0.465 0.0" rpy="0.0 0.0 0.0"/>
     <child link="left_wheel">left_wheel</child>
     <parent link="base_link">base_link</parent>
@@ -118,5 +118,5 @@
   </joint>
   <joint type="revolute" name="right_wheel_hinge">
-    <origin xyz="0.0 -0.2834 0.0" rpy="0.0 0.0 0.0"/>
+    <origin xyz="0.0 -0.465 0.0" rpy="0.0 0.0 0.0"/>
     <child link="right_wheel">right_wheel</child>
     <parent link="base_link">base_link</parent>

Commit message: apply format

File: igvc2023/urdf/orange.xacro (robot description, xacro)
@@ -1,17 +1,13 @@
 <?xml version="1.0"?>
 <!-- Revolute-Revolute Manipulator -->
-<robot name="orange" xmlns:xacro="http://www.ros.org/wiki/xacro">
+<robot xmlns:xacro="http://www.ros.org/wiki/xacro" name="orange">
   <!-- Constants for robot dimensions -->
   <xacro:property name="PI" value="3.1415926535897931"/>
   <!-- Macro -->
   <xacro:macro name="box_inertia" params="m x y z">
-    <inertia ixx="${m*(y*y+z*z)/12.0}" ixy = "0.0" ixz = "0.0"
-             iyy="${m*(z*z+x*x)/12.0}" iyz = "0.0"
-             izz="${m*(x*x+y*y)/12.0}" />
+    <inertia ixx="${m*(y*y+z*z)/12.0}" ixy="0.0" ixz="0.0" iyy="${m*(z*z+x*x)/12.0}" iyz="0.0" izz="${m*(x*x+y*y)/12.0}"/>
   </xacro:macro>
   <xacro:macro name="cylinder_inertia" params="m r h">
-    <inertia ixx="${m*(3*r*r+h*h)/12.0}" ixy = "0.0" ixz = "0.0"
-             iyy="${m*(3*r*r+h*h)/12.0}" iyz = "0.0"
-             izz="${m*r*r/2.0}" />
+    <inertia ixx="${m*(3*r*r+h*h)/12.0}" ixy="0.0" ixz="0.0" iyy="${m*(3*r*r+h*h)/12.0}" iyz="0.0" izz="${m*r*r/2.0}"/>
   </xacro:macro>
   <!-- Import gazebo reference -->
@@ -64,16 +60,16 @@
     </visual>
     <inertial>
-       <mass value="27.1" />
-       <origin xyz="-0.1995 0.0 0.19" rpy="0.0 0.0 0.0"/>
-       <xacro:box_inertia m="27.1" x="0.549" y="0.5055" z="0.3"/>
+      <mass value="27.1"/>
+      <origin xyz="-0.1995 0.0 0.19" rpy="0.0 0.0 0.0"/>
+      <xacro:box_inertia m="27.1" x="0.549" y="0.5055" z="0.3"/>
     </inertial>
   </link>
   <!-- Back wheels -->
-  <joint name="left_caster_hinge" type ="fixed">
+  <joint name="left_caster_hinge" type="fixed">
     <origin xyz="0.0 0.0 0.0" rpy="0.0 0.0 0.0"/>
     <child link="left_caster_link"/>
     <parent link="base_link"/>
   </joint>
-  <joint name="right_caster_hinge" type ="fixed">
+  <joint name="right_caster_hinge" type="fixed">
     <origin xyz="0.0 0.0 0.0" rpy="0.0 0.0 0.0"/>
     <child link="right_caster_link"/>
@@ -115,5 +111,5 @@
     <parent link="base_link">base_link</parent>
     <axis xyz="0 1 0"/>
-    <limit effort="100" velocity="100.0"  lower="-5000" upper="5000" />
+    <limit effort="100" velocity="100.0" lower="-5000" upper="5000"/>
   </joint>
   <joint type="revolute" name="right_wheel_hinge">
@@ -122,5 +118,5 @@
     <parent link="base_link">base_link</parent>
     <axis xyz="0 1 0"/>
-    <limit effort="100" velocity="100.0"  lower="-5000" upper="5000" />
+    <limit effort="100" velocity="100.0" lower="-5000" upper="5000"/>
   </joint>
   <link name="left_wheel">
@@ -138,7 +134,7 @@
     </visual>
     <inertial>
-       <mass value="3.4" />
-       <origin xyz="0.0 0.0 0.0" rpy="0.0 ${PI/2} ${PI/2}"/>
-       <xacro:cylinder_inertia m="3.4" r="0.1015" h="0.047"/>
+      <mass value="3.4"/>
+      <origin xyz="0.0 0.0 0.0" rpy="0.0 ${PI/2} ${PI/2}"/>
+      <xacro:cylinder_inertia m="3.4" r="0.1015" h="0.047"/>
     </inertial>
   </link>
@@ -157,7 +153,7 @@
     </visual>
     <inertial>
-       <mass value="3.4" />
-       <origin xyz="0.0 0.0 0.0" rpy="0.0 ${PI/2} ${PI/2}"/>
-       <xacro:cylinder_inertia m="3.4" r="0.1015" h="0.047"/>
+      <mass value="3.4"/>
+      <origin xyz="0.0 0.0 0.0" rpy="0.0 ${PI/2} ${PI/2}"/>
+      <xacro:cylinder_inertia m="3.4" r="0.1015" h="0.047"/>
     </inertial>
   </link>

File: igvc2023/urdf/sensors/camera.urdf.xacro (robot description, xacro)
@@ -1,6 +1,4 @@
 <?xml version="1.0"?>
-<robot name="sensor_camera" xmlns:xacro="http://ros.org/wiki/xacro"
-                            xmlns:controller="http://playerstage.sourceforge.net/gazebo/xmlschema/#controller"
-                            xmlns:interface="http://playerstage.sourceforge.net/gazebo/xmlschema/#interface">
+<robot xmlns:xacro="http://ros.org/wiki/xacro" xmlns:controller="http://playerstage.sourceforge.net/gazebo/xmlschema/#controller" xmlns:interface="http://playerstage.sourceforge.net/gazebo/xmlschema/#interface" name="sensor_camera">
   <xacro:property name="camera" value="0.1"/>
   <xacro:macro name="sensor_camera" params="name parent *origin">
@@ -65,3 +63,3 @@
     </gazebo>
   </xacro:macro>
- </robot>
+</robot>

File: igvc2023/urdf/sensors/gps.urdf.xacro (robot description, xacro)
@@ -1,12 +1,10 @@
 <?xml version="1.0"?>
-<robot name="sensor_gps" xmlns:xacro="http://ros.org/wiki/xacro"
-                         xmlns:controller="http://playerstage.sourceforge.net/gazebo/xmlschema/#controller"
-                         xmlns:interface="http://playerstage.sourceforge.net/gazebo/xmlschema/#interface">
+<robot xmlns:xacro="http://ros.org/wiki/xacro" xmlns:controller="http://playerstage.sourceforge.net/gazebo/xmlschema/#controller" xmlns:interface="http://playerstage.sourceforge.net/gazebo/xmlschema/#interface" name="sensor_gps">
   <xacro:macro name="sensor_gps" params="name parent *origin">
     <joint name="${name}_joint" type="fixed">
-        <xacro:insert_block name="origin"/>
-        <axis xyz="1 0 0"/>
-        <parent link="${parent}"/>
-        <child link="${name}_link"/>
+      <xacro:insert_block name="origin"/>
+      <axis xyz="1 0 0"/>
+      <parent link="${parent}"/>
+      <child link="${name}_link"/>
     </joint>
     <link name="${name}_link">
@@ -26,12 +24,12 @@
     <gazebo>
       <plugin name="gps" filename="libhector_gazebo_ros_gps.so">
-          <updateRate>1.0</updateRate>
-          <topicName>/fix</topicName>
-          <gaussianNoise>0.05 0.05 0.05</gaussianNoise>
-          <offset>0 0 0</offset>
-          <velocityGaussianNoise>0 0 0</velocityGaussianNoise>
-          <frameId>gps_link</frameId>
+        <updateRate>1.0</updateRate>
+        <topicName>/fix</topicName>
+        <gaussianNoise>0.05 0.05 0.05</gaussianNoise>
+        <offset>0 0 0</offset>
+        <velocityGaussianNoise>0 0 0</velocityGaussianNoise>
+        <frameId>gps_link</frameId>
       </plugin>
-     <material>Gazebo/White</material>
+      <material>Gazebo/White</material>
     </gazebo>
   </xacro:macro>

Commit message: Fix frame name and positions

File: igvc2023/urdf/orange.xacro (robot description, xacro)
@@ -35,5 +35,5 @@
   <xacro:include filename="$(find igvc2023)/urdf/sensors/camera.urdf.xacro"/>
   <xacro:sensor_camera name="camera" parent="base_link">
-    <origin xyz="0 0 1.3" rpy="0 ${PI/2} 0"/>
+    <origin xyz="0 0 1.3" rpy="0 0 0"/>
   </xacro:sensor_camera>
   <!-- Import gps model -->

File: igvc2023/urdf/sensors/camera.urdf.xacro (robot description, xacro)
@@ -29,5 +29,5 @@
         <update_rate>10.0</update_rate>
         <camera>
-          <pose>0 0 0 0 0 0</pose>
+          <pose>0 0 0 0 ${PI/2} 0</pose>
           <horizontal_fov>3.1415</horizontal_fov>
           <image>

Commit message: Change orange.xacro

File: igvc2023/urdf/orange.xacro (robot description, xacro)
@@ -52,7 +52,7 @@
   <link name="base_link">
     <collision>
-      <origin xyz="-0.6 0.0 0.5" rpy="0.0 0.0 0.0"/>
+      <origin xyz="-0.55 0.0 0.5" rpy="0.0 0.0 0.0"/>
       <geometry>
-        <box size="1.06 0.625 0.83"/>
+        <box size="1.6 0.85 1"/>
       </geometry>
     </collision>
@@ -82,5 +82,5 @@
   <link name="left_caster_link">
     <collision>
-      <origin xyz="-1.28015 0.15 -0.039" rpy="0.0 ${PI/2} ${PI/2}"/>
+      <origin xyz="-1.2015 0.15 -0.039" rpy="0.0 ${PI/2} ${PI/2}"/>
       <geometry>
         <sphere radius="0.0625"/>
