Commit message: Revert "apply format"
This reverts commit 93991a5f3df31227f23dc788c798bd9f2e6ec08e.

File: igvc2023/urdf/orange.xacro (robot description, xacro)
@@ -1,13 +1,17 @@
 <?xml version="1.0"?>
 <!-- Revolute-Revolute Manipulator -->
-<robot xmlns:xacro="http://www.ros.org/wiki/xacro" name="orange">
+<robot name="orange" xmlns:xacro="http://www.ros.org/wiki/xacro">
   <!-- Constants for robot dimensions -->
   <xacro:property name="PI" value="3.1415926535897931"/>
   <!-- Macro -->
   <xacro:macro name="box_inertia" params="m x y z">
-    <inertia ixx="${m*(y*y+z*z)/12.0}" ixy="0.0" ixz="0.0" iyy="${m*(z*z+x*x)/12.0}" iyz="0.0" izz="${m*(x*x+y*y)/12.0}"/>
+    <inertia ixx="${m*(y*y+z*z)/12.0}" ixy = "0.0" ixz = "0.0"
+             iyy="${m*(z*z+x*x)/12.0}" iyz = "0.0"
+             izz="${m*(x*x+y*y)/12.0}" />
   </xacro:macro>
   <xacro:macro name="cylinder_inertia" params="m r h">
-    <inertia ixx="${m*(3*r*r+h*h)/12.0}" ixy="0.0" ixz="0.0" iyy="${m*(3*r*r+h*h)/12.0}" iyz="0.0" izz="${m*r*r/2.0}"/>
+    <inertia ixx="${m*(3*r*r+h*h)/12.0}" ixy = "0.0" ixz = "0.0"
+             iyy="${m*(3*r*r+h*h)/12.0}" iyz = "0.0"
+             izz="${m*r*r/2.0}" />
   </xacro:macro>
   <!-- Import gazebo reference -->
@@ -60,16 +64,16 @@
     </visual>
     <inertial>
-      <mass value="27.1"/>
-      <origin xyz="-0.1995 0.0 0.19" rpy="0.0 0.0 0.0"/>
-      <xacro:box_inertia m="27.1" x="0.549" y="0.5055" z="0.3"/>
+       <mass value="27.1" />
+       <origin xyz="-0.1995 0.0 0.19" rpy="0.0 0.0 0.0"/>
+       <xacro:box_inertia m="27.1" x="0.549" y="0.5055" z="0.3"/>
     </inertial>
   </link>
   <!-- Back wheels -->
-  <joint name="left_caster_hinge" type="fixed">
+  <joint name="left_caster_hinge" type ="fixed">
     <origin xyz="0.0 0.0 0.0" rpy="0.0 0.0 0.0"/>
     <child link="left_caster_link"/>
     <parent link="base_link"/>
   </joint>
-  <joint name="right_caster_hinge" type="fixed">
+  <joint name="right_caster_hinge" type ="fixed">
     <origin xyz="0.0 0.0 0.0" rpy="0.0 0.0 0.0"/>
     <child link="right_caster_link"/>
@@ -111,5 +115,5 @@
     <parent link="base_link">base_link</parent>
     <axis xyz="0 1 0"/>
-    <limit effort="100" velocity="100.0" lower="-5000" upper="5000"/>
+    <limit effort="100" velocity="100.0"  lower="-5000" upper="5000" />
   </joint>
   <joint type="revolute" name="right_wheel_hinge">
@@ -118,5 +122,5 @@
     <parent link="base_link">base_link</parent>
     <axis xyz="0 1 0"/>
-    <limit effort="100" velocity="100.0" lower="-5000" upper="5000"/>
+    <limit effort="100" velocity="100.0"  lower="-5000" upper="5000" />
   </joint>
   <link name="left_wheel">
@@ -134,7 +138,7 @@
     </visual>
     <inertial>
-      <mass value="3.4"/>
-      <origin xyz="0.0 0.0 0.0" rpy="0.0 ${PI/2} ${PI/2}"/>
-      <xacro:cylinder_inertia m="3.4" r="0.1015" h="0.047"/>
+       <mass value="3.4" />
+       <origin xyz="0.0 0.0 0.0" rpy="0.0 ${PI/2} ${PI/2}"/>
+       <xacro:cylinder_inertia m="3.4" r="0.1015" h="0.047"/>
     </inertial>
   </link>
@@ -153,7 +157,7 @@
     </visual>
     <inertial>
-      <mass value="3.4"/>
-      <origin xyz="0.0 0.0 0.0" rpy="0.0 ${PI/2} ${PI/2}"/>
-      <xacro:cylinder_inertia m="3.4" r="0.1015" h="0.047"/>
+       <mass value="3.4" />
+       <origin xyz="0.0 0.0 0.0" rpy="0.0 ${PI/2} ${PI/2}"/>
+       <xacro:cylinder_inertia m="3.4" r="0.1015" h="0.047"/>
     </inertial>
   </link>

File: igvc2023/urdf/sensors/camera.urdf.xacro (robot description, xacro)
@@ -1,4 +1,6 @@
 <?xml version="1.0"?>
-<robot xmlns:xacro="http://ros.org/wiki/xacro" xmlns:controller="http://playerstage.sourceforge.net/gazebo/xmlschema/#controller" xmlns:interface="http://playerstage.sourceforge.net/gazebo/xmlschema/#interface" name="sensor_camera">
+<robot name="sensor_camera" xmlns:xacro="http://ros.org/wiki/xacro"
+                            xmlns:controller="http://playerstage.sourceforge.net/gazebo/xmlschema/#controller"
+                            xmlns:interface="http://playerstage.sourceforge.net/gazebo/xmlschema/#interface">
   <xacro:property name="camera" value="0.1"/>
   <xacro:macro name="sensor_camera" params="name parent *origin">
@@ -63,3 +65,3 @@
     </gazebo>
   </xacro:macro>
-</robot>
+ </robot>

File: igvc2023/urdf/sensors/gps.urdf.xacro (robot description, xacro)
@@ -1,10 +1,12 @@
 <?xml version="1.0"?>
-<robot xmlns:xacro="http://ros.org/wiki/xacro" xmlns:controller="http://playerstage.sourceforge.net/gazebo/xmlschema/#controller" xmlns:interface="http://playerstage.sourceforge.net/gazebo/xmlschema/#interface" name="sensor_gps">
+<robot name="sensor_gps" xmlns:xacro="http://ros.org/wiki/xacro"
+                         xmlns:controller="http://playerstage.sourceforge.net/gazebo/xmlschema/#controller"
+                         xmlns:interface="http://playerstage.sourceforge.net/gazebo/xmlschema/#interface">
   <xacro:macro name="sensor_gps" params="name parent *origin">
     <joint name="${name}_joint" type="fixed">
-      <xacro:insert_block name="origin"/>
-      <axis xyz="1 0 0"/>
-      <parent link="${parent}"/>
-      <child link="${name}_link"/>
+        <xacro:insert_block name="origin"/>
+        <axis xyz="1 0 0"/>
+        <parent link="${parent}"/>
+        <child link="${name}_link"/>
     </joint>
     <link name="${name}_link">
@@ -24,12 +26,12 @@
     <gazebo>
       <plugin name="gps" filename="libhector_gazebo_ros_gps.so">
-        <updateRate>1.0</updateRate>
-        <topicName>/fix</topicName>
-        <gaussianNoise>0.05 0.05 0.05</gaussianNoise>
-        <offset>0 0 0</offset>
-        <velocityGaussianNoise>0 0 0</velocityGaussianNoise>
-        <frameId>gps_link</frameId>
+          <updateRate>1.0</updateRate>
+          <topicName>/fix</topicName>
+          <gaussianNoise>0.05 0.05 0.05</gaussianNoise>
+          <offset>0 0 0</offset>
+          <velocityGaussianNoise>0 0 0</velocityGaussianNoise>
+          <frameId>gps_link</frameId>
       </plugin>
-      <material>Gazebo/White</material>
+     <material>Gazebo/White</material>
     </gazebo>
   </xacro:macro>

File: igvc2023/urdf/sensors/hokuyo.urdf.xacro (robot description, xacro)
@@ -1,9 +1,10 @@
 <?xml version="1.0"?>
-<robot xmlns:xacro="http://ros.org/wiki/xacro" xmlns:controller="http://playerstage.sourceforge.net/gazebo/xmlschema/#controller" xmlns:interface="http://playerstage.sourceforge.net/gazebo/xmlschema/#interface" name="sensor_hokuyo">
-  <xacro:property name="hokuyo_link" value="0.1"/>
-  <!-- Size of square 'hokuyo' box -->
+<robot name="sensor_hokuyo" xmlns:xacro="http://ros.org/wiki/xacro"
+                              xmlns:controller="http://playerstage.sourceforge.net/gazebo/xmlschema/#controller"
+                              xmlns:interface="http://playerstage.sourceforge.net/gazebo/xmlschema/#interface">
+  <xacro:property name="hokuyo_link" value="0.1" /> <!-- Size of square 'hokuyo' box -->
   <xacro:macro name="sensor_hokuyo" params="name parent *origin min_angle max_angle samples">
     <joint name="${name}_joint" type="fixed">
-      <xacro:insert_block name="origin"/>
+    	<xacro:insert_block name="origin"/>
       <axis xyz="0 1 0"/>
       <parent link="${parent}"/>
@@ -14,5 +15,5 @@
         <origin xyz="0 0 0" rpy="0 0 0"/>
         <geometry>
-          <box size="${hokuyo_link} ${hokuyo_link} ${hokuyo_link}"/>
+            <box size="${hokuyo_link} ${hokuyo_link} ${hokuyo_link}"/>
         </geometry>
       </collision>
@@ -30,38 +31,38 @@
     </link>
     <gazebo reference="hokuyo_link">
-      <sensor type="ray" name="head_hokuyo_sensor">
-        <pose>0 0 0 0 0 0</pose>
-        <visualize>false</visualize>
-        <update_rate>40</update_rate>
-        <ray>
-          <scan>
-            <horizontal>
-              <resolution>1</resolution>
-              <samples>${samples}</samples>
-              <min_angle>${min_angle}</min_angle>
-              <max_angle>${max_angle}</max_angle>
-            </horizontal>
-          </scan>
-          <range>
-            <min>0.10</min>
-            <max>30.0</max>
-            <resolution>0.01</resolution>
-          </range>
-          <noise>
-            <type>gaussian</type>
-            <!-- Noise parameters based on published spec for Hokuyo laser
+    <sensor type="ray" name="head_hokuyo_sensor">
+      <pose>0 0 0 0 0 0</pose>
+      <visualize>false</visualize>
+      <update_rate>40</update_rate>
+      <ray>
+        <scan>
+          <horizontal>
+            <resolution>1</resolution>
+            <samples>${samples}</samples>
+            <min_angle>${min_angle}</min_angle>
+            <max_angle>${max_angle}</max_angle>
+          </horizontal>
+        </scan>
+        <range>
+          <min>0.10</min>
+          <max>30.0</max>
+          <resolution>0.01</resolution>
+        </range>
+        <noise>
+          <type>gaussian</type>
+          <!-- Noise parameters based on published spec for Hokuyo laser
                achieving "+-30mm" accuracy at range < 10m.  A mean of 0.0m and
                stddev of 0.01m will put 99.7% of samples within 0.03m of the true
                reading. -->
-            <mean>0.0</mean>
-            <stddev>0.01</stddev>
-          </noise>
-        </ray>
-        <plugin name="gazebo_ros_head_hokuyo_controller" filename="libgazebo_ros_laser.so">
-          <topicName>/hokuyo_scan</topicName>
-          <frameName>hokuyo_link</frameName>
-        </plugin>
-      </sensor>
-    </gazebo>
+          <mean>0.0</mean>
+          <stddev>0.01</stddev>
+        </noise>
+      </ray>
+      <plugin name="gazebo_ros_head_hokuyo_controller" filename="libgazebo_ros_laser.so">
+        <topicName>/hokuyo_scan</topicName>
+        <frameName>hokuyo_link</frameName>
+      </plugin>
+    </sensor>
+  </gazebo>
   </xacro:macro>
 </robot>

File: igvc2023/urdf/sensors/imu.urdf.xacro (robot description, xacro)
@@ -1,29 +1,31 @@
 <?xml version="1.0"?>
-<robot xmlns:xacro="http://ros.org/wiki/xacro" xmlns:controller="http://playerstage.sourceforge.net/gazebo/xmlschema/#controller" xmlns:interface="http://playerstage.sourceforge.net/gazebo/xmlschema/#interface" name="sensor_imu">
+<robot name="sensor_imu" xmlns:xacro="http://ros.org/wiki/xacro"
+                         xmlns:controller="http://playerstage.sourceforge.net/gazebo/xmlschema/#controller"
+                         xmlns:interface="http://playerstage.sourceforge.net/gazebo/xmlschema/#interface">
   <xacro:macro name="sensor_imu" params="name parent *origin size">
     <joint name="${name}_joint" type="fixed">
-      <xacro:insert_block name="origin"/>
-      <axis xyz="1 0 0"/>
-      <parent link="${parent}"/>
-      <child link="${name}_link"/>
+        <xacro:insert_block name="origin"/>
+        <axis xyz="1 0 0"/>
+        <parent link="${parent}"/>
+        <child link="${name}_link"/>
     </joint>
     <link name="${name}_link">
-      <inertial>
-        <mass value="0.001"/>
-        <origin rpy="0 0 0" xyz="0 0 0"/>
-        <inertia ixx="0.0001" ixy="0" ixz="0" iyy="0.000001" iyz="0" izz="0.0001"/>
-      </inertial>
-      <visual>
-        <origin rpy="0 0 0" xyz="0 0 0"/>
-        <geometry>
-          <box size="${size}"/>
-        </geometry>
-      </visual>
-      <collision>
-        <origin rpy="0 0 0" xyz="0 0 0"/>
-        <geometry>
-          <box size="${size}"/>
-        </geometry>
-      </collision>
+        <inertial>
+          <mass value="0.001"/>
+          <origin rpy="0 0 0" xyz="0 0 0"/>
+          <inertia ixx="0.0001" ixy="0" ixz="0" iyy="0.000001" iyz="0" izz="0.0001"/>
+        </inertial>
+        <visual>
+          <origin rpy="0 0 0" xyz="0 0 0"/>
+          <geometry>
+            <box size="${size}"/>
+          </geometry>
+        </visual>
+        <collision>
+          <origin rpy="0 0 0" xyz="0 0 0"/>
+          <geometry>
+            <box size="${size}"/>
+          </geometry>
+        </collision>
     </link>
     <gazebo reference="${name}_link">
@@ -32,6 +34,5 @@
         <topic>imu</topic>
         <plugin name="imu_plugin" filename="libgazebo_ros_imu_sensor.so">
-          <bodyName>${name}_link</bodyName>
-          <!-- bodyName always set base_link by URDF parser -->
+          <bodyName>${name}_link</bodyName> <!-- bodyName always set base_link by URDF parser -->
           <frameName>${name}_link</frameName>
           <topicName>imu</topicName>

File: igvc2023/urdf/sensors/velodyne.urdf.xacro (robot description, xacro)
@@ -1,6 +1,7 @@
 <?xml version="1.0"?>
-<robot xmlns:xacro="http://ros.org/wiki/xacro" xmlns:controller="http://playerstage.sourceforge.net/gazebo/xmlschema/#controller" xmlns:interface="http://playerstage.sourceforge.net/gazebo/xmlschema/#interface" name="sensor_velodyne">
-  <xacro:property name="velodyne_link" value="0.1"/>
-  <!-- Size of square 'hokuyo' box -->
+<robot name="sensor_velodyne" xmlns:xacro="http://ros.org/wiki/xacro"
+                              xmlns:controller="http://playerstage.sourceforge.net/gazebo/xmlschema/#controller"
+                              xmlns:interface="http://playerstage.sourceforge.net/gazebo/xmlschema/#interface">
+  <xacro:property name="velodyne_link" value="0.1" /> <!-- Size of square 'hokuyo' box -->
   <xacro:macro name="sensor_velodyne" params="name parent *origin min_angle max_angle samples">
     <joint name="${name}_joint" type="fixed">
@@ -14,5 +15,5 @@
         <origin xyz="0 0 0" rpy="0 0 0"/>
         <geometry>
-          <box size="0.1 0.1 0.1"/>
+            <box size="0.1 0.1 0.1"/>
         </geometry>
       </collision>
